Commit message: moveit_controller수정, interface(multi_thread, fr3, demo.launch)추가

File: src/franka_description/robots/panda_arm.xacro (robot description, xacro)
@@ -45,5 +45,5 @@
         <origin xyz="0 0 -0.1915" rpy="0 0 0"/>
         <geometry>
-          <cylinder radius="${0.06+safety_distance}" length="0.2830" />
+          <cylinder radius="${0.05+safety_distance}" length="0.2830" />
         </geometry>
       </collision>
@@ -51,5 +51,5 @@
         <origin xyz="0 0 -0.333" rpy="0 0 0"/>
         <geometry>
-          <sphere radius="${0.06+safety_distance}" />
+          <sphere radius="${0.05+safety_distance}" />
         </geometry>
       </collision>
@@ -57,5 +57,5 @@
         <origin xyz="0 0 -0.05" rpy="0 0 0"/>
         <geometry>
-          <sphere radius="${0.06+safety_distance}" />
+          <sphere radius="${0.05+safety_distance}" />
         </geometry>
       </collision>
